File: ADS1292-breakout-kicad/eeg.kicad_pcb (KiCad board)
At the start: 2 copper layers, 31.6 x 24.8 mm, 29 parts, among them J1 Conn_01x02_Pin, J2 Conn_01x02_Pin, J3 Conn_01x02_Pin, J4 Conn_01x05_Pin, J5 Conn_01x01_Pin, U1 ADS1292IPBSR, U2 SP724AHTG

Commit message: updated pcb design
Parts:
- moved VCAP2-AVSS1 12.2 mm to (120.0, 87.0), turned to 180 degrees
- moved Vcap1-AVSS1 4.62 mm to (113.4, 103.4), turned to 90 degrees
- moved J2 2.21 mm to (107.2, 97.8)
- moved J1 2.05 mm to (104.7, 87.8)
- moved U2 1.70 mm to (106.2, 92.9)
- moved VREFP-AVSS#2 1.22 mm to (113.0, 100.0)
- moved VREFP-AVSS#1 1.22 mm to (114.6, 100.0)
- moved R1 0.80 mm to (121.4, 98.0)
- moved PGA2n-PGA2P1 0.42 mm to (113.1, 96.7)
- moved PGA1-PGA2 0.29 mm to (113.8, 89.7)
- moved H1 0.28 mm to (122.4, 102.6)
- moved R2 0.20 mm to (119.6, 99.2)
Routing:
- net Net-(U1-VCAP2): track 20.0 -> 4.29 mm
- net Net-(J3-Pin_2): track 64.0 -> 76.8 mm
- net Net-(U1-VCAP1): track 10.8 -> 7.51 mm
- net Net-(J2-Pin_2): track 15.7 -> 13.5 mm
- net Net-(J2-Pin_1): track 8.78 -> 6.88 mm
- net Net-(J3-Pin_1): track 39.7 -> 38.2 mm
- net Net-(J1-Pin_2): track 8.34 -> 6.99 mm
- net /PGA1_N: track 2.82 -> 1.81 mm
- net Net-(U1-START): track 4.22 -> 3.33 mm
- net Net-(U1-VREFP): track 5.13 -> 4.43 mm
- net Net-(J1-Pin_1): track 13.2 -> 13.8 mm
- net Net-(U1-*PWDN/*RESET): track 2.57 -> 3.11 mm
Other:
- board size 31.6 x 24.8 mm -> 25.4 x 22.2 mm
